File: datalogger v1.sch (EAGLE design)
At the start: 15 parts, among them M1 ARDUINO-NANO-3.0#ISP

Commit message: final
Parts:
- removed 12VIN, ADPT_GND, COMMON_GBD, JP1, JP2, REG_5V: (no value), pinhead:PINHD-1X1
- removed M1: ARDUINO-NANO-3.0#ISP, diy-modules:ARDUINO-NANO-3.0#ISP
- removed TO_WEMOS: (no value), pinhead:PINHD-1X4
- added 5V_REGS: (no value), pinhead:PINHD-1X2
- added 5V_REG_DUST, 5V_REG_WEMOS: (no value), pinhead:PINHD-1X1
- added LCD: (no value), pinhead:PINHD-1X4
- added LUX: (no value), adafruit:PINHD-1X3
- added M2: ARDUINO-NANO-3.0, diy-modules:ARDUINO-NANO-3.0
- added U$1: MP1584, MP1584-dc-brick:MP1584
- added U$2: WEMOS-D1-MINI, diy-modules:WEMOS-D1-MINI
- added U$3: EDGE_CONNECTOR, P_Dusk:EDGE_CONNECTOR
- added X1: (no value), power-jack:DC-2.1MM-5MM
Connections:
- removed net 12V_ADP: 12VIN.1, M1.VIN
- new net 12V: M2.VIN, U$1.VIN+, U$3.12V, X1.3
- new net D_THERMO: M2.D9, THERMOCOUPLE.5
- new net LUX_A: LUX.1, M2.A0
- new net SCL_LCD: LCD.1, U$2.D1
- new net SDA_LCD: LCD.2, U$2.D2
- net 5V: now also LUX.2, SGP30.1; no longer JP1.1, JP2.1, SGP30.2, WSP2110.2
- net 5V_REG: now also 5V_REGS.1, 5V_REGS.2, 5V_REG_DUST.1, 5V_REG_WEMOS.1, LCD.3, U$1.VOUT+, U$2.5V, U$3.5V, WSP2110.2; no longer REG_5V.1, TO_WEMOS.1
- net CLK: now also M2.D13/SCK; no longer M1.D13/SCK
- net CS: now also M2.D10; no longer M1.D10
- net CS_THERMO: now also M2.D8; no longer M1.D9
- net DATA-DHT22: now also DHT22.3, M2.D4; no longer DHT22.2, M1.D4
- net GND: now also DHT22.2, LCD.4, LUX.3, M2.GND.1, SGP30.2, U$1.VOUT-, U$2.GND; no longer COMMON_GBD.1, DHT22.3, M1.GND.1, SGP30.1, TO_WEMOS.2
- net GND_ADP: now also M2.GND.2, U$1.VIN-, U$3.GND, X1.2; no longer ADPT_GND.1, M1.GND.2
- net MISO: now also M2.D11/MOSI; no longer M1.D11/MOSI
- net MOSI: now also M2.D12/MISO; no longer M1.D12/MISO, THERMOCOUPLE.5
- net RX_WEMOS: now also M2.D1/TX, U$2.RX; no longer M1.D1/TX, TO_WEMOS.3
- net SCL: now also M2.A5; no longer M1.A5
- net SDA: now also M2.A4; no longer M1.A4
- net SIG: now also M2.A3; no longer M1.A3
- net TX_WEMOS: now also M2.D0/RX, U$2.TX; no longer M1.D0/RX, TO_WEMOS.4
- net VOUT-1: now also M2.D2; no longer M1.D2
- net VOUT-2: now also M2.D3; no longer M1.D3

Commit message: update
Connections:
- net MISO: now also M2.D12/MISO; no longer M2.D11/MOSI
- net MOSI: now also M2.D11/MOSI; no longer M2.D12/MISO
Changed lines of the file:
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@@
 </segment>
 <segment>
-<wire x1="2.54" y1="73.66" x2="-10.16" y2="73.66" width="0.1524" layer="91"/>
-<label x="-10.16" y="73.66" size="1.778" layer="95"/>
-<pinref part="M2" gate="G$1" pin="D11/MOSI"/>
+<pinref part="M2" gate="G$1" pin="D12/MISO"/>
+<wire x1="2.54" y1="71.12" x2="-10.16" y2="71.12" width="0.1524" layer="91"/>
+<label x="-10.16" y="71.12" size="1.778" layer="95"/>
 </segment>
 </net>
@@
 </segment>
 <segment>
-<wire x1="2.54" y1="71.12" x2="-10.16" y2="71.12" width="0.1524" layer="91"/>
-<label x="-10.16" y="71.12" size="1.778" layer="95"/>
-<pinref part="M2" gate="G$1" pin="D12/MISO"/>
+<pinref part="M2" gate="G$1" pin="D11/MOSI"/>
+<wire x1="2.54" y1="73.66" x2="-10.16" y2="73.66" width="0.1524" layer="91"/>
+<label x="-10.16" y="73.66" size="1.778" layer="95"/>
 </segment>
 </net>

Commit message: update board
Parts:
- added U$4, U$5: JUMP-NO, P_Dusk:JUMP-NO
Connections:
- new net N$2: 5V_REG_WEMOS.1, LCD.3, U$2.5V, U$4.J1
- net 5V: now also U$4.J2, U$5.J2
- net 5V_REG: now also U$5.J1; no longer 5V_REG_WEMOS.1, LCD.3, U$2.5V
Other:
- moved on the sheet: 5V_REG_DUST
Changed lines of the file:
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@@
 <part name="X1" library="power-jack" deviceset="DC" device="-5MM" technology="-2.1MM"/>
 <part name="5V_REGS" library="pinhead" library_urn="urn:adsk.eagle:library:325" deviceset="PINHD-1X2" device="" package3d_urn="urn:adsk.eagle:package:22435/2"/>
+<part name="U$4" library="P_Dusk" deviceset="JUMP-NO" device=""/>
+<part name="U$5" library="P_Dusk" deviceset="JUMP-NO" device=""/>
 </parts>
 <sheets>
@@
 <attribute name="VALUE" x="89.408" y="105.156" size="1.778" layer="96"/>
 </instance>
-<instance part="5V_REG_DUST" gate="G$1" x="114.3" y="-5.08" smashed="yes">
-<attribute name="NAME" x="107.95" y="-1.905" size="1.778" layer="95"/>
-<attribute name="VALUE" x="107.95" y="-10.16" size="1.778" layer="96"/>
+<instance part="5V_REG_DUST" gate="G$1" x="119.38" y="-5.08" smashed="yes">
+<attribute name="NAME" x="113.03" y="-1.905" size="1.778" layer="95"/>
+<attribute name="VALUE" x="113.03" y="-10.16" size="1.778" layer="96"/>
 </instance>
 <instance part="M2" gate="G$1" x="22.86" y="88.9" smashed="yes">
@@
 <attribute name="VALUE" x="-13.97" y="-35.56" size="1.778" layer="96"/>
 </instance>
+<instance part="U$4" gate="G$1" x="40.64" y="15.24" smashed="yes">
+<attribute name="NAME" x="43.18" y="22.86" size="1.778" layer="94"/>
+</instance>
+<instance part="U$5" gate="G$1" x="119.38" y="-17.78" smashed="yes">
+<attribute name="NAME" x="121.92" y="-10.16" size="1.778" layer="94"/>
+</instance>
 </instances>
 <busses>
@@
 <label x="76.2" y="17.78" size="1.778" layer="95"/>
 </segment>
+<segment>
+<wire x1="132.08" y1="-15.24" x2="144.78" y2="-15.24" width="0.1524" layer="91"/>
+<label x="141.478" y="-14.986" size="1.778" layer="95"/>
+<pinref part="U$5" gate="G$1" pin="J2"/>
+</segment>
+<segment>
+<wire x1="53.34" y1="17.78" x2="60.96" y2="17.78" width="0.1524" layer="91"/>
+<label x="58.42" y="17.78" size="1.778" layer="95"/>
+<pinref part="U$4" gate="G$1" pin="J2"/>
+</segment>
 </net>
 <net name="DATA-DHT22" class="0">
@@
 <pinref part="U$2" gate="G$1" pin="GND"/>
 <wire x1="2.54" y1="25.4" x2="17.78" y2="25.4" width="0.1524" layer="91"/>
-<label x="7.62" y="25.4" size="1.778" layer="95"/>
+<label x="12.7" y="25.4" size="1.778" layer="95"/>
 </segment>
 <segment>
 <pinref part="LCD" gate="A" pin="4"/>
-<wire x1="33.274" y1="27.94" x2="15.24" y2="27.94" width="0.1524" layer="91"/>
-<label x="15.24" y="27.94" size="1.778" layer="95"/>
+<wire x1="33.274" y1="27.94" x2="22.86" y2="27.94" width="0.1524" layer="91"/>
+<label x="22.86" y="27.94" size="1.778" layer="95"/>
 </segment>
 <segment>
@@
 <label x="76.2" y="-5.08" size="1.778" layer="95"/>
 <pinref part="5V_REG_DUST" gate="G$1" pin="1"/>
-<wire x1="93.98" y1="-5.08" x2="111.76" y2="-5.08" width="0.1524" layer="91"/>
+<wire x1="93.98" y1="-5.08" x2="106.68" y2="-5.08" width="0.1524" layer="91"/>
 <junction x="93.98" y="-5.08"/>
-</segment>
-<segment>
-<pinref part="U$2" gate="G$1" pin="5V"/>
-<wire x1="2.54" y1="22.86" x2="15.24" y2="22.86" width="0.1524" layer="91"/>
-<label x="7.62" y="22.86" size="1.778" layer="95"/>
-<pinref part="5V_REG_WEMOS" gate="G$1" pin="1"/>
-<wire x1="15.24" y1="22.86" x2="17.78" y2="22.86" width="0.1524" layer="91"/>
-<wire x1="17.78" y1="5.08" x2="15.24" y2="5.08" width="0.1524" layer="91"/>
-<wire x1="15.24" y1="5.08" x2="-4.064" y2="5.08" width="0.1524" layer="91"/>
-<wire x1="15.24" y1="22.86" x2="15.24" y2="5.08" width="0.1524" layer="91"/>
-<junction x="15.24" y="5.08"/>
-</segment>
-<segment>
-<pinref part="LCD" gate="A" pin="3"/>
-<wire x1="33.274" y1="30.48" x2="15.24" y2="30.48" width="0.1524" layer="91"/>
-<label x="15.24" y="30.48" size="1.778" layer="95"/>
+<wire x1="106.68" y1="-5.08" x2="116.84" y2="-5.08" width="0.1524" layer="91"/>
+<wire x1="121.92" y1="-15.24" x2="106.68" y2="-15.24" width="0.1524" layer="91"/>
+<wire x1="106.68" y1="-15.24" x2="106.68" y2="-5.08" width="0.1524" layer="91"/>
+<junction x="106.68" y="-5.08"/>
+<pinref part="U$5" gate="G$1" pin="J1"/>
 </segment>
 <segment>
@@
 </segment>
 </net>
+<net name="N$2" class="0">
+<segment>
+<pinref part="U$2" gate="G$1" pin="5V"/>
+<wire x1="2.54" y1="22.86" x2="10.16" y2="22.86" width="0.1524" layer="91"/>
+<wire x1="10.16" y1="22.86" x2="10.16" y2="17.78" width="0.1524" layer="91"/>
+<pinref part="5V_REG_WEMOS" gate="G$1" pin="1"/>
+<wire x1="10.16" y1="17.78" x2="10.16" y2="5.08" width="0.1524" layer="91"/>
+<wire x1="10.16" y1="5.08" x2="-4.064" y2="5.08" width="0.1524" layer="91"/>
+<wire x1="43.18" y1="17.78" x2="20.32" y2="17.78" width="0.1524" layer="91"/>
+<junction x="10.16" y="17.78"/>
+<pinref part="LCD" gate="A" pin="3"/>
+<wire x1="20.32" y1="17.78" x2="10.16" y2="17.78" width="0.1524" layer="91"/>
+<wire x1="33.274" y1="30.48" x2="20.32" y2="30.48" width="0.1524" layer="91"/>
+<wire x1="20.32" y1="30.48" x2="20.32" y2="17.78" width="0.1524" layer="91"/>
+<junction x="20.32" y="17.78"/>
+<pinref part="U$4" gate="G$1" pin="J1"/>
+</segment>
+</net>

Commit message: update pcb
Connections:
- net 5V: now also DHT22.2; no longer DHT22.1
- net GND: now also DHT22.1; no longer DHT22.2
Changed lines of the file:
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@@
 <net name="5V" class="0">
-<segment>
-<pinref part="DHT22" gate="A" pin="1"/>
-<wire x1="93.98" y1="71.12" x2="76.2" y2="71.12" width="0.1524" layer="91"/>
-<label x="76.2" y="71.12" size="1.778" layer="95"/>
-</segment>
 <segment>
 <pinref part="RTC" gate="A" pin="2"/>
@@
 <label x="58.42" y="17.78" size="1.778" layer="95"/>
 <pinref part="U$4" gate="G$1" pin="J2"/>
+</segment>
+<segment>
+<pinref part="DHT22" gate="A" pin="2"/>
+<wire x1="93.98" y1="68.58" x2="76.2" y2="68.58" width="0.1524" layer="91"/>
+<label x="76.2" y="68.58" size="1.778" layer="95"/>
 </segment>
 </net>
@@
 </segment>
 <segment>
-<pinref part="DHT22" gate="A" pin="2"/>
-<wire x1="93.98" y1="68.58" x2="76.2" y2="68.58" width="0.1524" layer="91"/>
-<label x="76.2" y="68.58" size="1.778" layer="95"/>
+<pinref part="DHT22" gate="A" pin="1"/>
+<wire x1="93.98" y1="71.12" x2="76.2" y2="71.12" width="0.1524" layer="91"/>
+<label x="76.2" y="71.12" size="1.778" layer="95"/>
 </segment>
 </net>

Commit message: update
Parts:
- removed LUX: (no value), adafruit:PINHD-1X3
- removed U$4, U$5: JUMP-NO, P_Dusk:JUMP-NO
- added FAN-HD: (no value), pinhead:PINHD-1X2
- added LUX_A: (no value), pinhead:PINHD-1X3
- added NO-JUMP-PAD2, NO-JUMP_PAD: JUMP-NO, P_Dusk:JUMP-NO
- renumbered 5V_REG_DUST to 5V_REG
Connections:
- removed net N$1: DSM501A.1
- net 12V: now also FAN-HD.1
- net 5V: now also LUX_A.2, M2.5V, NO-JUMP-PAD2.J2, NO-JUMP_PAD.J2; no longer LUX.2, U$4.J2, U$5.J2
- net 5V_REG: now also NO-JUMP-PAD2.J1; no longer U$5.J1
- net GND: now also LUX_A.3; no longer LUX.3
- net GND_ADP: now also FAN-HD.2
- net LUX_A: now also LUX_A.1; no longer LUX.1
- net N$2: now also NO-JUMP_PAD.J1; no longer U$4.J1
Other:
- moved on the sheet: 5V_REGS, 5V_REG_WEMOS
